Commit message: Add Usagi robot launch and description files
- Introduced view_robot.launch.py for launching Usagi robot components including robot_state_publisher, joint_state_publisher_gui, and RViz.
- Updated CMakeLists.txt to include additional directories for meshes and RViz configurations.
- Added multiple STL mesh files for Usagi robot components (arms, body, cups, wheels).
- Created usagi.rviz configuration file for visualizing the Usagi robot in RViz.
- Added URDF and Xacro files for the Usagi robot, defining its structure and joint configurations.

File: usagi_description/urdf/usagi.urdf (robot description, URDF)
Before this commit: robot usagi, 12 links, 11 joints
Joints:
- joint base_link_to_usagi_body: limit lower=-3.14159 upper=3.14159 effort=${joint_effort} velocity=${joint_velocity} -> lower=-3.14159 upper=3.14159 effort=1.37 velocity=7.0; type fixed -> revolute
- joint usagi_arm1_to_usagi_cup1: limit lower=-3.14159 upper=3.14159 effort=0.0 velocity=${joint_velocity} -> lower=-3.14159 upper=3.14159 effort=1.37 velocity=7.0
- joint usagi_arm2_to_usagi_cup2: limit lower=-3.14159 upper=3.14159 effort=0.0 velocity=${joint_velocity} -> lower=-3.14159 upper=3.14159 effort=1.37 velocity=7.0
- joint usagi_arm3_to_usagi_cup3: limit lower=-3.14159 upper=3.14159 effort=0.0 velocity=${joint_velocity} -> lower=-3.14159 upper=3.14159 effort=1.37 velocity=7.0
- joint usagi_arm4_to_usagi_cup4: limit lower=-3.14159 upper=3.14159 effort=0.0 velocity=${joint_velocity} -> lower=-3.14159 upper=3.14159 effort=1.37 velocity=7.0
- joint usagi_body_to_usagi_arm1: limit lower=-3.14159 upper=3.14159 effort=${joint_effort} velocity=${joint_velocity} -> lower=-3.14159 upper=3.14159 effort=1.37 velocity=7.0
- joint usagi_body_to_usagi_arm2: limit lower=-3.14159 upper=3.14159 effort=${joint_effort} velocity=${joint_velocity} -> lower=-3.14159 upper=3.14159 effort=1.37 velocity=7.0
- joint usagi_body_to_usagi_arm3: limit lower=-3.14159 upper=3.14159 effort=${joint_effort} velocity=${joint_velocity} -> lower=-3.14159 upper=3.14159 effort=1.37 velocity=7.0
- joint usagi_body_to_usagi_arm4: limit lower=-3.14159 upper=3.14159 effort=${joint_effort} velocity=${joint_velocity} -> lower=-3.14159 upper=3.14159 effort=1.37 velocity=7.0
- joint usagi_body_to_usagi_wheel1: limit lower=-3.14159 upper=3.14159 effort=${joint_effort} velocity=${joint_velocity} -> lower=-3.14159 upper=3.14159 effort=1.37 velocity=7.0
- joint usagi_body_to_usagi_wheel2: limit lower=-3.14159 upper=3.14159 effort=${joint_effort} velocity=${joint_velocity} -> lower=-3.14159 upper=3.14159 effort=1.37 velocity=7.0
